Commit message: adding a grasping frame with a fixed/revolute joint

File: romeo_description/urdf/romeo_generated_urdf/romeo_arms.xacro (robot description, xacro)
@@ -107,6 +107,18 @@
 		<xacro:insert_visu_l_wrist/>
 	</link>
+	<joint name="LGrasp" type="revolute">
+		<parent link="l_wrist"/>
+		<child link="l_grasp_link"/>
+		<origin rpy="0 0 0" xyz="0.065 0.0 0.0"/>
+		<limit effort="0.0" lower="0" upper="0.0" velocity="0.0"/>
+	</joint>
+	<link name="l_grasp_link">
+		<inertial>
+			<mass value="0"/>
+			<inertia ixx="0" ixy="0" ixz="0" iyy="0" iyz="0" izz="0"/>
+		</inertial>
+	</link>
 	<joint name="LHand" type="revolute">
-		<parent link="l_wrist"/>
+		<parent link="l_grasp_link"/>
 		<child link="l_gripper"/>
 		<origin rpy="1.5708 0.0450146 -3.14159" xyz="-0.0579412 -0.0159 -0.00260997"/>
@@ -223,6 +235,18 @@
 		<xacro:insert_visu_r_wrist/>
 	</link>
+	<joint name="RGrasp" type="revolute">
+		<parent link="r_wrist"/>
+		<child link="r_grasp_link"/>
+		<origin rpy="0 0 0" xyz="0.065 0.0 0.0"/>
+		<limit effort="0.0" lower="0" upper="0.0" velocity="0.0"/>
+	</joint>
+	<link name="r_grasp_link">
+		<inertial>
+			<mass value="0"/>
+			<inertia ixx="0" ixy="0" ixz="0" iyy="0" iyz="0" izz="0"/>
+		</inertial>
+	</link>
 	<joint name="RHand" type="revolute">
-		<parent link="r_wrist"/>
+		<parent link="r_grasp_link"/>
 		<child link="r_gripper"/>
 		<origin rpy="1.5708 0.0450146 -3.14159" xyz="-0.0579412 -0.0159 -0.00260997"/>
